File: hardware/pqfp_80_64nixie/pqfp_80_64nixie.sch (KiCad schematic (older format))
At the start: 88 parts, among them J1 Conn_01x16, J2 Conn_01x16, J3 Conn_01x16, J4 Conn_01x16, J5 Conn_01x16, J6 NK01B, J7 Screw_Terminal_01x02, U1 PQFP-80

Commit message: Fixing NK01B pinout
Connections:
- net GND: now also J6.1 (Pin_1), J6.7 (Pin_7); no longer J6.2 (Pin_2), J6.8 (Pin_8)
- net PULSE: now also J6.6 (Pin_6); no longer J6.3 (Pin_3)
- net RX: now also J6.3 (Pin_3); no longer J6.6 (Pin_6)
- net VIN: now also J6.8 (Pin_8); no longer J6.1 (Pin_1)
- net VOUT: now also J6.4 (Pin_4); no longer J6.5 (Pin_5)
Changed lines of the file:
@@
 L Connector_Generic:Conn_01x08 J6
 U 1 1 5E408107
-P 800 7250
-F 0 "J6" H 718 6625 50  0000 C CNN
-F 1 "NK01B" H 718 6716 50  0000 C CNN
-F 2 "Connector_PinSocket_2.54mm:PinSocket_1x08_P2.54mm_Vertical" H 800 7250 50  0001 C CNN
-F 3 "https://threeneurons.wordpress.com/nixie-power-supply/hv-supply-kit/" H 800 7250 50  0001 C CNN
-	1    800  7250
-	-1   0    0    1
+P 800 7150
+F 0 "J6" H 718 6525 50  0000 C CNN
+F 1 "NK01B" H 718 6616 50  0000 C CNN
+F 2 "Connector_PinSocket_2.54mm:PinSocket_1x08_P2.54mm_Vertical" H 800 7150 50  0001 C CNN
+F 3 "https://threeneurons.wordpress.com/nixie-power-supply/hv-supply-kit/" H 800 7150 50  0001 C CNN
+	1    800  7150
+	-1   0    0    -1
 $EndComp
 Wire Wire Line
